File: philoctetes.kicad_sch (KiCad schematic)
At the start: 174 parts, among them U2 TRRS

Commit message: added case files
Parts:
- DL1, DL10, DL11, DL12, DL13, DL14, DL15, DL16, DL17, DL18, DL19, DL2, DL20, DL21, DL3, DL4, DL5, DL6, DL7, DL8, DL9: renamed from DL?; footprint Diode_SMD:D_SOD-323 -> Diode_SMD:D_SOD-323_HandSoldering
- L1, L10, L11, L12, L13, L14, L15, L16, L17, L18, L19, L2, L20, L21, L3, L4, L5, L6, L7, L8, L9: renamed from L?; footprint mysuperawesomekb:Hotswap_Choc_V1V2_1.00u -> philoctetes:Hotswap_Choc_V1V2_1.00u
- LEDU_L1, LEDU_L2, LEDU_L3, LEDU_L4, LEDU_L5, LEDU_L6: renamed from LEDU_L?; footprint mysuperawesomekb:LED_SK6812MINI-E_faceup -> philoctetes:LED_SK6812MINI-E_faceup; symbol home:SK6821MINI-E_faceup -> philoctetes:SK6821MINI-E_faceup
- LEDU_R1: footprint mysuperawesomekb:LED_SK6812MINI-E_faceup -> philoctetes:LED_SK6812MINI-E_faceup; symbol home:SK6821MINI-E_faceup -> philoctetes:SK6821MINI-E_faceup
- LEDU_R2: renamed from LEDU_R6; footprint mysuperawesomekb:LED_SK6812MINI-E_faceup -> philoctetes:LED_SK6812MINI-E_faceup; symbol home:SK6821MINI-E_faceup -> philoctetes:SK6821MINI-E_faceup
- LEDU_R3: renamed from LEDU_R2; footprint mysuperawesomekb:LED_SK6812MINI-E_faceup -> philoctetes:LED_SK6812MINI-E_faceup; symbol home:SK6821MINI-E_faceup -> philoctetes:SK6821MINI-E_faceup
- LEDU_R4: renamed from LEDU_R5; footprint mysuperawesomekb:LED_SK6812MINI-E_faceup -> philoctetes:LED_SK6812MINI-E_faceup; symbol home:SK6821MINI-E_faceup -> philoctetes:SK6821MINI-E_faceup
- LEDU_R5: renamed from LEDU_R3; footprint mysuperawesomekb:LED_SK6812MINI-E_faceup -> philoctetes:LED_SK6812MINI-E_faceup; symbol home:SK6821MINI-E_faceup -> philoctetes:SK6821MINI-E_faceup
- LEDU_R6: renamed from LEDU_R4; footprint mysuperawesomekb:LED_SK6812MINI-E_faceup -> philoctetes:LED_SK6812MINI-E_faceup; symbol home:SK6821MINI-E_faceup -> philoctetes:SK6821MINI-E_faceup
- LED_L1, LED_L10, LED_L11, LED_L12, LED_L13, LED_L14, LED_L15, LED_L16, LED_L17, LED_L18, LED_L19, LED_L2, LED_L20, LED_L21, LED_L3, LED_L4, LED_L5, LED_L6, LED_L7, LED_L8, LED_L9: renamed from LED_L?; footprint mysuperawesomekb:LED_SK6812MINI-E_facedown -> philoctetes:LED_SK6812MINI-E_facedown; symbol home:SK6821MINI-E_facedown -> philoctetes:SK6821MINI-E_facedown
- LED_R1: renamed from LED_R10; footprint mysuperawesomekb:LED_SK6812MINI-E_facedown -> philoctetes:LED_SK6812MINI-E_facedown; symbol home:SK6821MINI-E_facedown -> philoctetes:SK6821MINI-E_facedown
- LED_R10: renamed from LED_R17; footprint mysuperawesomekb:LED_SK6812MINI-E_facedown -> philoctetes:LED_SK6812MINI-E_facedown; symbol home:SK6821MINI-E_facedown -> philoctetes:SK6821MINI-E_facedown
- LED_R11: renamed from LED_R16; footprint mysuperawesomekb:LED_SK6812MINI-E_facedown -> philoctetes:LED_SK6812MINI-E_facedown; symbol home:SK6821MINI-E_facedown -> philoctetes:SK6821MINI-E_facedown
- LED_R12: renamed from LED_R15; footprint mysuperawesomekb:LED_SK6812MINI-E_facedown -> philoctetes:LED_SK6812MINI-E_facedown; symbol home:SK6821MINI-E_facedown -> philoctetes:SK6821MINI-E_facedown
- LED_R13: renamed from LED_R19; footprint mysuperawesomekb:LED_SK6812MINI-E_facedown -> philoctetes:LED_SK6812MINI-E_facedown; symbol home:SK6821MINI-E_facedown -> philoctetes:SK6821MINI-E_facedown
- LED_R14: renamed from LED_R20; footprint mysuperawesomekb:LED_SK6812MINI-E_facedown -> philoctetes:LED_SK6812MINI-E_facedown; symbol home:SK6821MINI-E_facedown -> philoctetes:SK6821MINI-E_facedown
- LED_R15: renamed from LED_R21; footprint mysuperawesomekb:LED_SK6812MINI-E_facedown -> philoctetes:LED_SK6812MINI-E_facedown; symbol home:SK6821MINI-E_facedown -> philoctetes:SK6821MINI-E_facedown
- LED_R16: renamed from LED_R24; footprint mysuperawesomekb:LED_SK6812MINI-E_facedown -> philoctetes:LED_SK6812MINI-E_facedown; symbol home:SK6821MINI-E_facedown -> philoctetes:SK6821MINI-E_facedown
- LED_R17: renamed from LED_R23; footprint mysuperawesomekb:LED_SK6812MINI-E_facedown -> philoctetes:LED_SK6812MINI-E_facedown; symbol home:SK6821MINI-E_facedown -> philoctetes:SK6821MINI-E_facedown
- LED_R18: renamed from LED_R22; footprint mysuperawesomekb:LED_SK6812MINI-E_facedown -> philoctetes:LED_SK6812MINI-E_facedown; symbol home:SK6821MINI-E_facedown -> philoctetes:SK6821MINI-E_facedown
- LED_R19: renamed from LED_R25; footprint mysuperawesomekb:LED_SK6812MINI-E_facedown -> philoctetes:LED_SK6812MINI-E_facedown; symbol home:SK6821MINI-E_facedown -> philoctetes:SK6821MINI-E_facedown
- LED_R2: renamed from LED_R9; footprint mysuperawesomekb:LED_SK6812MINI-E_facedown -> philoctetes:LED_SK6812MINI-E_facedown; symbol home:SK6821MINI-E_facedown -> philoctetes:SK6821MINI-E_facedown
- LED_R20: renamed from LED_R26; footprint mysuperawesomekb:LED_SK6812MINI-E_facedown -> philoctetes:LED_SK6812MINI-E_facedown; symbol home:SK6821MINI-E_facedown -> philoctetes:SK6821MINI-E_facedown
- LED_R21: renamed from LED_R27; footprint mysuperawesomekb:LED_SK6812MINI-E_facedown -> philoctetes:LED_SK6812MINI-E_facedown; symbol home:SK6821MINI-E_facedown -> philoctetes:SK6821MINI-E_facedown
- LED_R3: renamed from LED_R8; footprint mysuperawesomekb:LED_SK6812MINI-E_facedown -> philoctetes:LED_SK6812MINI-E_facedown; symbol home:SK6821MINI-E_facedown -> philoctetes:SK6821MINI-E_facedown
- LED_R4: renamed from LED_R7; footprint mysuperawesomekb:LED_SK6812MINI-E_facedown -> philoctetes:LED_SK6812MINI-E_facedown; symbol home:SK6821MINI-E_facedown -> philoctetes:SK6821MINI-E_facedown
- LED_R5: renamed from LED_R11; footprint mysuperawesomekb:LED_SK6812MINI-E_facedown -> philoctetes:LED_SK6812MINI-E_facedown; symbol home:SK6821MINI-E_facedown -> philoctetes:SK6821MINI-E_facedown
- LED_R6: renamed from LED_R12; footprint mysuperawesomekb:LED_SK6812MINI-E_facedown -> philoctetes:LED_SK6812MINI-E_facedown; symbol home:SK6821MINI-E_facedown -> philoctetes:SK6821MINI-E_facedown
- LED_R7: renamed from LED_R13; footprint mysuperawesomekb:LED_SK6812MINI-E_facedown -> philoctetes:LED_SK6812MINI-E_facedown; symbol home:SK6821MINI-E_facedown -> philoctetes:SK6821MINI-E_facedown
- LED_R8: renamed from LED_R14; footprint mysuperawesomekb:LED_SK6812MINI-E_facedown -> philoctetes:LED_SK6812MINI-E_facedown; symbol home:SK6821MINI-E_facedown -> philoctetes:SK6821MINI-E_facedown
- LED_R9: renamed from LED_R18; footprint mysuperawesomekb:LED_SK6812MINI-E_facedown -> philoctetes:LED_SK6812MINI-E_facedown; symbol home:SK6821MINI-E_facedown -> philoctetes:SK6821MINI-E_facedown
- LEFT1: renamed from LEFT?; footprint mysuperawesomekb:nice_nano_AH_USBup -> philoctetes:nice_nano_AH_USBup
- PSW1: renamed from PSW?; footprint totem:MSK12C02 -> philoctetes:MSK12C02
- PSW2: renamed from PSW1; footprint totem:MSK12C02 -> philoctetes:MSK12C02
- R10: renamed from R4; footprint mysuperawesomekb:Hotswap_Choc_V1V2_1.00u -> philoctetes:Hotswap_Choc_V1V2_1.00u
- R11: renamed from R10; footprint mysuperawesomekb:Hotswap_Choc_V1V2_1.00u -> philoctetes:Hotswap_Choc_V1V2_1.00u
- R12: renamed from R16; footprint mysuperawesomekb:Hotswap_Choc_V1V2_1.00u -> philoctetes:Hotswap_Choc_V1V2_1.00u
- R13: renamed from R19; footprint mysuperawesomekb:Hotswap_Choc_V1V2_1.00u -> philoctetes:Hotswap_Choc_V1V2_1.00u
- R14: renamed from R3; footprint mysuperawesomekb:Hotswap_Choc_V1V2_1.00u -> philoctetes:Hotswap_Choc_V1V2_1.00u
- R15: renamed from R9; footprint mysuperawesomekb:Hotswap_Choc_V1V2_1.00u -> philoctetes:Hotswap_Choc_V1V2_1.00u
- R16: renamed from R15; footprint mysuperawesomekb:Hotswap_Choc_V1V2_1.00u -> philoctetes:Hotswap_Choc_V1V2_1.00u
- R17: renamed from R2; footprint mysuperawesomekb:Hotswap_Choc_V1V2_1.00u -> philoctetes:Hotswap_Choc_V1V2_1.00u
- R18: renamed from R8; footprint mysuperawesomekb:Hotswap_Choc_V1V2_1.00u -> philoctetes:Hotswap_Choc_V1V2_1.00u
- R19: renamed from R14; footprint mysuperawesomekb:Hotswap_Choc_V1V2_1.00u -> philoctetes:Hotswap_Choc_V1V2_1.00u
- R2: renamed from R6; footprint mysuperawesomekb:Hotswap_Choc_V1V2_1.00u -> philoctetes:Hotswap_Choc_V1V2_1.00u
- R20: renamed from R1; footprint mysuperawesomekb:Hotswap_Choc_V1V2_1.00u -> philoctetes:Hotswap_Choc_V1V2_1.00u
- R21: renamed from R7; footprint mysuperawesomekb:Hotswap_Choc_V1V2_1.00u -> philoctetes:Hotswap_Choc_V1V2_1.00u
- R22: renamed from R13; footprint mysuperawesomekb:Hotswap_Choc_V1V2_1.00u -> philoctetes:Hotswap_Choc_V1V2_1.00u
- R3: renamed from R12; footprint mysuperawesomekb:Hotswap_Choc_V1V2_1.00u -> philoctetes:Hotswap_Choc_V1V2_1.00u
- R4: renamed from R18; footprint mysuperawesomekb:Hotswap_Choc_V1V2_1.00u -> philoctetes:Hotswap_Choc_V1V2_1.00u
- R5: renamed from R21; footprint mysuperawesomekb:Hotswap_Choc_V1V2_1.00u -> philoctetes:Hotswap_Choc_V1V2_1.00u
- R6: renamed from R5; footprint mysuperawesomekb:Hotswap_Choc_V1V2_1.00u -> philoctetes:Hotswap_Choc_V1V2_1.00u
- R7: renamed from R11; footprint mysuperawesomekb:Hotswap_Choc_V1V2_1.00u -> philoctetes:Hotswap_Choc_V1V2_1.00u
- R8: renamed from R17; footprint mysuperawesomekb:Hotswap_Choc_V1V2_1.00u -> philoctetes:Hotswap_Choc_V1V2_1.00u
- R9: renamed from R20; footprint mysuperawesomekb:Hotswap_Choc_V1V2_1.00u -> philoctetes:Hotswap_Choc_V1V2_1.00u
- RIGHT1: footprint mysuperawesomekb:nice_nano_AH_USBup -> philoctetes:nice_nano_AH_USBup
- SW_NO_L1: renamed from SW_NO_L?; footprint mysuperawesomekb:SW_RST -> philoctetes:SW_RST
- SW_NO_R1: footprint mysuperawesomekb:SW_RST -> philoctetes:SW_RST
- U1: renamed from U?; footprint mysuperawesomekb:TRRS_PJ-320A -> philoctetes:TRRS_PJ-320A
- U2: footprint mysuperawesomekb:TRRS_PJ-320A -> philoctetes:TRRS_PJ-320A
- view_L1: renamed from view_L?; footprint mysuperawesomekb:nice_view -> philoctetes:nice_view
- view_R1: footprint mysuperawesomekb:nice_view -> philoctetes:nice_view
- gave numbers to parts that had none: 13
- renumbered BT1 to BT2, CR3 to CR1, CR1 to CR3, D6 to D1, D16 to D11, D19 to D12, D3 to D13, D9 to D14, D2 to D16, D8 to D17, D14 to D18, D1 to D19, D12 to D2, D7 to D20, D13 to D21, D18 to D3, D21 to D4, D11 to D6, D17 to D7, D20 to D8, D4 to D9, H_RIGHT6 to H_RIGHT1, H_RIGHT7 to H_RIGHT2, H_RIGHT8 to H_RIGHT3, H_RIGHT5 to H_RIGHT4, H_RIGHT3 to H_RIGHT5, H_RIGHT4 to H_RIGHT6, H_RIGHT2 to H_RIGHT7, H_RIGHT1 to H_RIGHT8

Commit message: updates annotations
Parts:
- DL1: footprint Diode_SMD:D_SOD-323_HandSoldering -> Diode_SMD:D_SOD-123F
- renumbered D19 to D1, D6 to D11, D2 to D12, D21 to D13, D18 to D14, D11 to D16, D7 to D17, D3 to D18, D12 to D19, D16 to D2, D8 to D20, D4 to D21, D13 to D3, D9 to D4, D1 to D6, D20 to D7, D17 to D8, D14 to D9, DL11 to DL10, DL15 to DL11, DL19 to DL12, DL3 to DL13, DL6 to DL14, DL9 to DL15, DL12 to DL16, DL16 to DL17, DL20 to DL18, DL13 to DL19, DL4 to DL2, DL17 to DL20, DL7 to DL3, DL10 to DL4, DL14 to DL5, DL18 to DL6, DL2 to DL7, DL5 to DL8, DL8 to DL9, H_RIGHT8 to H_RIGHT1, H_RIGHT7 to H_RIGHT2, H_RIGHT5 to H_RIGHT3, H_RIGHT6 to H_RIGHT4, H_RIGHT4 to H_RIGHT5, H_RIGHT3 to H_RIGHT6, H_RIGHT1 to H_RIGHT7, H_RIGHT2 to H_RIGHT8, RDOWN1 to R2, LEDU_L1 to led1, LED_L10 to led10, LED_L14 to led11, LED_L18 to led12, LED_L2 to led13, LED_L5 to led14, LED_L8 to led15, LED_L15 to led16, LED_L19 to led17, LED_L11 to led18, LED_L3 to led19, LEDU_L3 to led2, LED_L6 to led20, LED_L9 to led21, LED_L12 to led22, LED_L16 to led23, LED_L20 to led24, LED_L13 to led25, LED_L17 to led26, LED_L21 to led27, LEDU_R5 to led28, LEDU_R3 to led29, LEDU_L5 to led3, LEDU_R1 to led30, LEDU_R6 to led31, LEDU_R4 to led32, LEDU_R2 to led33, LED_R19 to led34, LED_R16 to led35, LED_R13 to led36, LED_R9 to led37, LED_R5 to led38, LED_R1 to led39, LEDU_L2 to led4, LED_R20 to led40, LED_R17 to led41, LED_R14 to led42, LED_R10 to led43, LED_R6 to led44, LED_R2 to led45, LED_R21 to led46, LED_R18 to led47, LED_R15 to led48, LED_R11 to led49, LEDU_L4 to led5, LED_R7 to led50, LED_R3 to led51, LED_R12 to led52, LED_R8 to led53, LED_R4 to led54, LEDU_L6 to led6, LED_L1 to led7, LED_L4 to led8, LED_L7 to led9, L1 to sw1, L11 to sw10, L15 to sw11, L19 to sw12, L3 to sw13, L6 to sw14, L9 to sw15, L12 to sw16, L16 to sw17, L20 to sw18, L13 to sw19, L4 to sw2, L17 to sw20, L21 to sw21, R20 to sw22, R17 to sw23, R14 to sw24, R10 to sw25, R6 to sw26, R2 to sw27, R21 to sw28, R18 to sw29, L7 to sw3, R15 to sw30, R11 to sw31, R7 to sw32, R3 to sw33, R22 to sw34, R19 to sw35, R16 to sw36, R12 to sw37, R8 to sw38, R4 to sw39, L10 to sw4, R13 to sw40, R9 to sw41, R5 to sw42, L14 to sw5, L18 to sw6, L2 to sw7, L5 to sw8, L8 to sw9, view_L1 to view1, view_R1 to view2
Other:
- moved on the sheet: D1, D10, D11, D12, D13, D14, D15, D16, D17, D18, D19, D2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
