File: PCBs/base_template/philoctetes.kicad_pcb (KiCad board)
At the start: 2 copper layers, 336.3 x 122.1 mm, 174 parts, among them U1 TRRS, U2 TRRS, sw1 Keyswitch, sw10 Keyswitch, sw11 Keyswitch, sw12 Keyswitch, sw13 Keyswitch, sw14 Keyswitch, sw15 Keyswitch, sw16 Keyswitch, sw17 Keyswitch, sw18 Keyswitch, sw19 Keyswitch, sw2 Keyswitch, sw20 Keyswitch, sw21 Keyswitch, sw22 Keyswitch, sw23 Keyswitch, sw24 Keyswitch, sw25 Keyswitch, sw26 Keyswitch, sw27 Keyswitch, sw28 Keyswitch, sw29 Keyswitch, sw3 Keyswitch, sw30 Keyswitch, sw31 Keyswitch, sw32 Keyswitch, sw33 Keyswitch, sw34 Keyswitch, sw35 Keyswitch, sw36 Keyswitch, sw37 Keyswitch, sw38 Keyswitch, sw39 Keyswitch, sw4 Keyswitch, sw40 Keyswitch, sw41 Keyswitch, sw42 Keyswitch, sw5 Keyswitch, sw6 Keyswitch, sw7 Keyswitch, sw8 Keyswitch, sw9 Keyswitch

Commit message: layout right side improvements
Parts:
- added BT_Cut1: Battery_Cut_12x37mm, philoctetes:Battery_Cut_12x37mm, F.Cu at (217.2, 189.0)
- added BT_Cut2: Battery_Cut_12x37mm, philoctetes:Battery_Cut_12x37mm, F.Cu at (252.5, 82.0)
- CL3, CR3: footprint Capacitor_SMD:CP_Elec_5x5.4 -> philoctetes:CP_Radial_D5.0mm_P2.00mm
- D1, D10, D11, D12, D13, D14, D15, D16, D17, D18, D19, D2, D20, D21, D3, D4, D5, D6, D7, D8, D9: footprint Diode_SMD:D_SOD-323 -> Diode_SMD:D_SOD-123F
- DL1, DL10, DL11, DL12, DL13, DL14, DL15, DL16, DL17, DL18, DL19, DL2, DL20, DL21, DL3, DL4, DL5, DL6, DL7, DL8, DL9: footprint Diode_SMD:D_SOD-323_HandSoldering -> Diode_SMD:D_SOD-123F
- moved sw22 104.7 mm to (379.7, 86.1), turned to 170.59 degrees
- moved sw27 103.9 mm to (275.5, 69.0), turned to 180 degrees
- moved sw28 102.0 mm to (376.7, 104.9), turned to 170.59 degrees
- moved sw33 100.8 mm to (275.5, 88.0), turned to 180 degrees
- moved sw34 98.7 mm to (373.5, 123.5), turned to 170.59 degrees
- moved sw39 97.3 mm to (275.5, 106.9), turned to 180 degrees
- moved sw23 67.2 mm to (360.7, 83.0), turned to 170.59 degrees
- moved sw26 66.1 mm to (294.5, 69.0), turned to 180 degrees
- moved sw29 64.2 mm to (357.7, 101.5), turned to 170.59 degrees
- moved sw32 62.8 mm to (294.8, 88.0), turned to 180 degrees
- moved sw35 61.3 mm to (354.6, 120.4), turned to 170.59 degrees
- moved sw38 59.3 mm to (294.8, 107.0), turned to 180 degrees
- moved sw42 47.3 mm to (243.7, 145.1), turned to -147.76 degrees
- moved sw40 47.0 mm to (288.8, 131.2), turned to 180 degrees
- moved sw25 25.0 mm to (315.2, 60.5), turned to 180 degrees
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Routing:
- removed copper zone on B.Cu, net GND_R
- removed copper zone on F.Cu, net GND_R
Other:
- board size 336.3 x 122.1 mm -> 336.7 x 122.1 mm

Commit message: working on routing
Parts:
- moved H_RIGHT7 169.4 mm to (108.0, 233.5)
- moved H_RIGHT8 169.4 mm to (116.0, 234.0)
- moved H_LEFT8 132.8 mm to (148.1, 235.2)
- moved H_LEFT7 132.8 mm to (134.5, 235.2)
- moved BT_Cut1 108.2 mm to (202.9, 81.7)
- moved R1 15.2 mm to (194.6, 91.8), turned to -90 degrees
- moved SW_NO_L1 13.8 mm to (211.4, 95.8), turned to -90 degrees
- moved D9 12.6 mm to (322.4, 83.4)
- moved H_LEFT6 11.8 mm to (65.0, 84.8)
- moved view1 11.5 mm to (196.0, 111.0)
- moved H_LEFT5 10.6 mm to (115.2, 120.6)
- moved CL2 8.25 mm to (199.3, 61.3), turned to 180 degrees
- moved CL1 8.15 mm to (205.2, 61.2), turned to 180 degrees
- moved BT1 7.45 mm to (196.0, 104.5), turned to 90 degrees
- moved led4 7.10 mm to (121.5, 116.4)
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Routing:
- net GND_R: track 0.00 -> 737.4 mm, vias 0 -> 24
- net +3.3V_R: track 0.00 -> 604.4 mm
- net row3_R: track 0.00 -> 77.8 mm, vias 0 -> 2
- net row2_R: track 0.00 -> 67.7 mm, vias 0 -> 4
- net Net-(D21-A): track 0.00 -> 55.6 mm
- net col2_R: track 0.00 -> 45.2 mm, vias 0 -> 2
- net col1_R: track 0.00 -> 43.4 mm
- net col6_R: track 0.00 -> 39.0 mm, vias 0 -> 4
- net Net-(led36-DOUT): track 0.00 -> 35.1 mm
- net row1_R: track 0.00 -> 34.9 mm, vias 0 -> 4
- net Net-(D20-A): track 0.00 -> 29.5 mm
- net Net-(led28-DOUT): track 0.00 -> 27.4 mm, vias 0 -> 2
- net Net-(led31-DOUT): track 0.00 -> 20.2 mm, vias 0 -> 2
- net Net-(D6-A): track 0.00 -> 17.9 mm
- net Net-(led29-DIN): track 0.00 -> 13.3 mm
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- removed copper zone on B.Cu, net GND_L
- removed copper zone on F.Cu, net GND_L
Other:
- board size 336.7 x 122.1 mm -> 336.3 x 122.1 mm

Commit message: routing right half; diodes, power, reset, tx, rx, clk...
Parts:
- CR1, CR2, R2: moved to B.Cu
- moved CR2 39.8 mm to (264.6, 98.7), turned to -90 degrees
- moved CR1 38.7 mm to (267.1, 98.6), turned to -90 degrees
- moved R2 26.4 mm to (242.6, 72.8), turned to 90 degrees
- moved led25 2.00 mm to (166.8, 128.4)
- moved led26 2.00 mm to (190.7, 130.8)
- moved led27 2.00 mm to (214.4, 142.8)
- moved led53 2.00 mm to (264.8, 131.0)
- moved led54 2.00 mm to (241.1, 143.2)
- moved sw19 2.00 mm to (166.9, 133.3)
- moved sw20 2.00 mm to (189.5, 135.6)
- moved sw21 2.00 mm to (211.7, 147.0)
- moved sw40 2.00 mm to (288.8, 133.2)
- moved sw41 2.00 mm to (265.9, 135.6)
- moved sw42 2.00 mm to (243.7, 147.1)
- moved led52 2.00 mm to (288.7, 128.5)
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Connections:
- R2 pad 1: Net-(RIGHT1-P0-10-LF) -> Net-(RIGHT1-P0.20)
- RIGHT1 pad 10: row2_R -> LED_R
- RIGHT1 pad 23: Net-(RIGHT1-P0-10-LF) -> row1_R
- RIGHT1 pad 24: unconnected-(RIGHT1-P0.09-LF-Pad24) -> row2_R
- RIGHT1 pad 5: SLA_R -> unconnected-(RIGHT1-P0.17-Pad5)
- RIGHT1 pad 6: SDA_R -> Net-(RIGHT1-P0.20)
- RIGHT1 pad 7: LED_R -> SLA_R
- RIGHT1 pad 8: CS_R -> SDA_R
- RIGHT1 pad 9: row1_R -> CS_R
Routing:
- net GND_R: track 737.4 -> 932.1 mm, vias 24 -> 32
- net col1_R: track 43.4 -> 213.0 mm, vias 0 -> 1
- net col3_R: track 0.00 -> 153.1 mm, vias 0 -> 7
- net col5_R: track 0.00 -> 145.9 mm, vias 0 -> 9
- net col2_R: track 45.2 -> 187.2 mm, vias 2 -> 5
- net col4_R: track 0.00 -> 139.8 mm, vias 0 -> 9
- net row1_R: track 34.9 -> 149.3 mm, vias 4 -> 9
- net row3_R: track 77.8 -> 180.8 mm, vias 2 -> 5
- net row2_R: track 67.7 -> 151.8 mm, vias 4 -> 11
- net col6_R: track 39.0 -> 119.9 mm, vias 4 -> 10
- net Net-(BT2-+): track 0.00 -> 69.3 mm
- net LED_R: track 0.00 -> 62.2 mm, vias 0 -> 2
- net row4_R: track 7.35 -> 60.6 mm, vias 0 -> 3
- net TX_R: track 0.00 -> 51.7 mm, vias 0 -> 1
- net RESET_R: track 0.00 -> 49.7 mm, vias 0 -> 1
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Other:
- outline, holes or cut-outs redrawn
